File: project/5v_power_supply.kicad_sch (KiCad schematic)
At the start: 6 parts, among them SW1 SW_5V, U3 TPS61235P

Commit message: Final revision
Parts:
- renumbered C8 to C7, C10 to C8, R10 to R5
Changed lines of the file:
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@@
   (symbol (lib_id "power:GND") (at 143.51 110.49 0) (unit 1)
     (in_bom yes) (on_board yes) (dnp no) (fields_autoplaced)
-    (property "Reference" "#PWR04" (at 143.51 116.84 0)
+    (property "Reference" "#PWR011" (at 143.51 116.84 0)
       (effects (font (size 1.27 1.27)) hide)
     )
@@
     (instances
       (project "picoups"
-        (path "/d62f1157-7c2f-4dce-8167-d5624900d267"
-          (reference "#PWR04") (unit 1)
-        )
         (path "/d62f1157-7c2f-4dce-8167-d5624900d267/92ed0473-53e9-4211-a651-f912f1c2bd2b"
           (reference "#PWR011") (unit 1)
@@
   (symbol (lib_id "power:GND") (at 109.22 101.6 0) (unit 1)
     (in_bom yes) (on_board yes) (dnp no) (fields_autoplaced)
-    (property "Reference" "#PWR021" (at 109.22 107.95 0)
+    (property "Reference" "#PWR019" (at 109.22 107.95 0)
       (effects (font (size 1.27 1.27)) hide)
     )
@@
     (instances
       (project "picoups"
-        (path "/d62f1157-7c2f-4dce-8167-d5624900d267"
-          (reference "#PWR021") (unit 1)
-        )
         (path "/d62f1157-7c2f-4dce-8167-d5624900d267/92ed0473-53e9-4211-a651-f912f1c2bd2b"
           (reference "#PWR019") (unit 1)
@@
   (symbol (lib_id "Device:C") (at 109.22 95.25 0) (unit 1)
     (in_bom yes) (on_board yes) (dnp no) (fields_autoplaced)
-    (property "Reference" "C8" (at 113.03 93.98 0)
+    (property "Reference" "C7" (at 113.03 93.98 0)
       (effects (font (size 1.27 1.27)) (justify left))
     )
@@
     (instances
       (project "picoups"
-        (path "/d62f1157-7c2f-4dce-8167-d5624900d267"
-          (reference "C8") (unit 1)
-        )
         (path "/d62f1157-7c2f-4dce-8167-d5624900d267/92ed0473-53e9-4211-a651-f912f1c2bd2b"
           (reference "C7") (unit 1)
@@
     (instances
       (project "picoups"
-        (path "/d62f1157-7c2f-4dce-8167-d5624900d267"
-          (reference "#PWR017") (unit 1)
-        )
         (path "/d62f1157-7c2f-4dce-8167-d5624900d267/92ed0473-53e9-4211-a651-f912f1c2bd2b"
           (reference "#PWR017") (unit 1)
@@
     (instances
       (project "picoups"
-        (path "/d62f1157-7c2f-4dce-8167-d5624900d267"
+        (path "/d62f1157-7c2f-4dce-8167-d5624900d267/92ed0473-53e9-4211-a651-f912f1c2bd2b"
           (reference "U3") (unit 1)
         )
-        (path "/d62f1157-7c2f-4dce-8167-d5624900d267/92ed0473-53e9-4211-a651-f912f1c2bd2b"
-          (reference "U3") (unit 1)
-        )
       )
     )
@@
     (instances
       (project "picoups"
-        (path "/d62f1157-7c2f-4dce-8167-d5624900d267"
+        (path "/d62f1157-7c2f-4dce-8167-d5624900d267/92ed0473-53e9-4211-a651-f912f1c2bd2b"
           (reference "L2") (unit 1)
         )
-        (path "/d62f1157-7c2f-4dce-8167-d5624900d267/92ed0473-53e9-4211-a651-f912f1c2bd2b"
-          (reference "L2") (unit 1)
-        )
       )
     )
@@
     (instances
       (project "picoups"
-        (path "/d62f1157-7c2f-4dce-8167-d5624900d267"
+        (path "/d62f1157-7c2f-4dce-8167-d5624900d267/92ed0473-53e9-4211-a651-f912f1c2bd2b"
           (reference "#PWR018") (unit 1)
         )
-        (path "/d62f1157-7c2f-4dce-8167-d5624900d267/92ed0473-53e9-4211-a651-f912f1c2bd2b"
-          (reference "#PWR018") (unit 1)
-        )
       )
     )
@@
     (instances
       (project "picoups"
-        (path "/d62f1157-7c2f-4dce-8167-d5624900d267"
+        (path "/d62f1157-7c2f-4dce-8167-d5624900d267/92ed0473-53e9-4211-a651-f912f1c2bd2b"
           (reference "SW1") (unit 1)
         )
-        (path "/d62f1157-7c2f-4dce-8167-d5624900d267/92ed0473-53e9-4211-a651-f912f1c2bd2b"
-          (reference "SW1") (unit 1)
-        )
       )
     )
@@
   (symbol (lib_id "power:GND") (at 185.42 101.6 0) (unit 1)
     (in_bom yes) (on_board yes) (dnp no) (fields_autoplaced)
-    (property "Reference" "#PWR022" (at 185.42 107.95 0)
+    (property "Reference" "#PWR021" (at 185.42 107.95 0)
       (effects (font (size 1.27 1.27)) hide)
     )
@@
     (instances
       (project "picoups"
-        (path "/d62f1157-7c2f-4dce-8167-d5624900d267"
-          (reference "#PWR022") (unit 1)
-        )
         (path "/d62f1157-7c2f-4dce-8167-d5624900d267/92ed0473-53e9-4211-a651-f912f1c2bd2b"
           (reference "#PWR021") (unit 1)
@@
   (symbol (lib_id "power:GND") (at 143.51 87.63 180) (unit 1)
     (in_bom yes) (on_board yes) (dnp no) (fields_autoplaced)
-    (property "Reference" "#PWR019" (at 143.51 81.28 0)
+    (property "Reference" "#PWR04" (at 143.51 81.28 0)
       (effects (font (size 1.27 1.27)) hide)
     )
@@
     (instances
       (project "picoups"
-        (path "/d62f1157-7c2f-4dce-8167-d5624900d267"
-          (reference "#PWR019") (unit 1)
-        )
         (path "/d62f1157-7c2f-4dce-8167-d5624900d267/92ed0473-53e9-4211-a651-f912f1c2bd2b"
           (reference "#PWR04") (unit 1)
@@
   (symbol (lib_id "Device:R") (at 143.51 102.87 180) (unit 1)
     (in_bom yes) (on_board yes) (dnp no)
-    (property "Reference" "R10" (at 139.7 101.6 0)
+    (property "Reference" "R5" (at 139.7 101.6 0)
       (effects (font (size 1.27 1.27)))
     )
@@
     (instances
       (project "picoups"
-        (path "/d62f1157-7c2f-4dce-8167-d5624900d267"
-          (reference "R10") (unit 1)
-        )
         (path "/d62f1157-7c2f-4dce-8167-d5624900d267/92ed0473-53e9-4211-a651-f912f1c2bd2b"
           (reference "R5") (unit 1)
@@
   (symbol (lib_id "Device:C") (at 185.42 95.25 0) (unit 1)
     (in_bom yes) (on_board yes) (dnp no) (fields_autoplaced)
-    (property "Reference" "C10" (at 189.23 93.98 0)
+    (property "Reference" "C8" (at 189.23 93.98 0)
       (effects (font (size 1.27 1.27)) (justify left))
     )
@@
     (instances
       (project "picoups"
-        (path "/d62f1157-7c2f-4dce-8167-d5624900d267"
-          (reference "C10") (unit 1)
-        )
         (path "/d62f1157-7c2f-4dce-8167-d5624900d267/92ed0473-53e9-4211-a651-f912f1c2bd2b"
           (reference "C8") (unit 1)
