File: project/picoups.kicad_sch (KiCad schematic)
At the start: 16 parts, among them J1 VIN, J2 BATT, J3 USB_C_Receptacle, J4 Conn_02x20_Odd_Even, Q1 Q_PMOS_GSD, SW2 SW_USER, U6 M41T62

Commit message: Minor improvements
Parts:
- added TP3: 5V, TestPoint:TestPoint_Pad_D1.0mm, symbol Connector:TestPoint
- added TP4, TP5: GND, TestPoint:TestPoint_Pad_D1.0mm, symbol Connector:TestPoint
- added TP6, TP8: VBAT, TestPoint:TestPoint_Pad_D1.0mm, symbol Connector:TestPoint
Connections:
- net 5V: now also TP3.1
- net GND: now also TP4.1, TP5.1
- net VBAT+: now also TP6.1
- net VBAT_SOL-: now also TP8.1
Changed lines of the file:
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@@
+    (stroke (width 0) (type default))
+  )
+  (wire (pts (xy 189.23 92.71) (xy 189.23 95.25))
     (stroke (width 0) (type default))
   )
@@
     (stroke (width 0) (type default))
   )
+  (wire (pts (xy 180.34 92.71) (xy 180.34 95.25))
+    (stroke (width 0) (type default))
+  )
   (wire (pts (xy 60.96 35.56) (xy 60.96 38.1))
     (stroke (width 0) (type default))
@@
     (stroke (width 0) (type default))
   )
+  (wire (pts (xy 207.01 92.71) (xy 207.01 95.25))
+    (stroke (width 0) (type default))
+  )
   (wire (pts (xy 49.53 30.48) (xy 49.53 26.67))
     (stroke (width 0) (type default))
@@
     (stroke (width 0) (type default))
   )
+  (wire (pts (xy 198.12 92.71) (xy 198.12 95.25))
+    (stroke (width 0) (type default))
+  )
   (wire (pts (xy 195.58 76.2) (xy 199.39 76.2))
     (stroke (width 0) (type default))
@@
   )
   (wire (pts (xy 139.7 52.07) (xy 143.51 52.07))
+    (stroke (width 0) (type default))
+  )
+  (wire (pts (xy 215.9 92.71) (xy 215.9 95.25))
     (stroke (width 0) (type default))
   )
@@
     )
   )
+  (global_label "VBAT+" (shape passive) (at 198.12 95.25 270) (fields_autoplaced)
+    (effects (font (size 1.27 1.27)) (justify right))
+    (property "Intersheetrefs" "${INTERSHEET_REFS}" (at 198.12 103.1111 90)
+      (effects (font (size 1.27 1.27)) (justify right) hide)
+    )
+  )
   (global_label "VBAT-" (shape passive) (at 143.51 99.06 0) (fields_autoplaced)
     (effects (font (size 1.27 1.27)) (justify left))
@@
     )
   )
+  (global_label "5V-" (shape passive) (at 215.9 95.25 270) (fields_autoplaced)
+    (effects (font (size 1.27 1.27)) (justify right))
+    (property "Intersheetrefs" "${INTERSHEET_REFS}" (at 215.9 100.9944 90)
+      (effects (font (size 1.27 1.27)) (justify right) hide)
+    )
+  )
   (global_label "SCL" (shape bidirectional) (at 127 109.22 270) (fields_autoplaced)
     (effects (font (size 1.27 1.27)) (justify right))
     (property "Intersheetrefs" "${INTERSHEET_REFS}" (at 127 116.7447 90)
       (effects (font (size 1.27 1.27)) (justify left) hide)
+    )
+  )
+  (global_label "VBAT_SOL-" (shape passive) (at 180.34 95.25 270) (fields_autoplaced)
+    (effects (font (size 1.27 1.27)) (justify right))
+    (property "Intersheetrefs" "${INTERSHEET_REFS}" (at 180.34 107.6468 90)
+      (effects (font (size 1.27 1.27)) (justify right) hide)
     )
   )
@@
         (path "/d62f1157-7c2f-4dce-8167-d5624900d267"
           (reference "#PWR029") (unit 1)
+        )
+      )
+    )
+  )
+  (symbol (lib_id "Connector:TestPoint") (at 215.9 92.71 0) (unit 1)
+    (in_bom yes) (on_board yes) (dnp no) (fields_autoplaced)
+    (property "Reference" "TP3" (at 218.44 88.138 0)
+      (effects (font (size 1.27 1.27)) (justify left))
+    )
+    (property "Value" "5V" (at 218.44 90.678 0)
+      (effects (font (size 1.27 1.27)) (justify left))
+    )
+    (property "Footprint" "TestPoint:TestPoint_Pad_D1.0mm" (at 220.98 92.71 0)
+      (effects (font (size 1.27 1.27)) hide)
+    )
+    (property "Datasheet" "~" (at 220.98 92.71 0)
+      (effects (font (size 1.27 1.27)) hide)
+    )
+    (pin "1")
+    (instances
+      (project "picoups"
+        (path "/d62f1157-7c2f-4dce-8167-d5624900d267"
+          (reference "TP3") (unit 1)
+        )
+        (path "/d62f1157-7c2f-4dce-8167-d5624900d267/69257c21-ade6-4c01-a27c-653d8ba74447"
+          (reference "TP2") (unit 1)
         )
       )
@@
     )
   )
+  (symbol (lib_id "Connector:TestPoint") (at 189.23 92.71 0) (unit 1)
+    (in_bom yes) (on_board yes) (dnp no)
+    (property "Reference" "TP5" (at 191.77 88.138 0)
+      (effects (font (size 1.27 1.27)) (justify left))
+    )
+    (property "Value" "GND" (at 191.77 90.678 0)
+      (effects (font (size 1.27 1.27)) (justify left))
+    )
+    (property "Footprint" "TestPoint:TestPoint_Pad_D1.0mm" (at 194.31 92.71 0)
+      (effects (font (size 1.27 1.27)) hide)
+    )
+    (property "Datasheet" "~" (at 194.31 92.71 0)
+      (effects (font (size 1.27 1.27)) hide)
+    )
+    (pin "1")
+    (instances
+      (project "picoups"
+        (path "/d62f1157-7c2f-4dce-8167-d5624900d267"
+          (reference "TP5") (unit 1)
+        )
+        (path "/d62f1157-7c2f-4dce-8167-d5624900d267/69257c21-ade6-4c01-a27c-653d8ba74447"
+          (reference "TP2") (unit 1)
+        )
+      )
+    )
+  )
   (symbol (lib_id "Connector_Generic:Conn_01x02") (at 207.01 24.13 270) (mirror x) (unit 1)
     (in_bom yes) (on_board yes) (dnp no)
@@
     )
   )
+  (symbol (lib_id "Connector:TestPoint") (at 207.01 92.71 0) (unit 1)
+    (in_bom yes) (on_board yes) (dnp no)
+    (property "Reference" "TP4" (at 209.55 88.138 0)
+      (effects (font (size 1.27 1.27)) (justify left))
+    )
+    (property "Value" "GND" (at 209.55 90.678 0)
+      (effects (font (size 1.27 1.27)) (justify left))
+    )
+    (property "Footprint" "TestPoint:TestPoint_Pad_D1.0mm" (at 212.09 92.71 0)
+      (effects (font (size 1.27 1.27)) hide)
+    )
+    (property "Datasheet" "~" (at 212.09 92.71 0)
+      (effects (font (size 1.27 1.27)) hide)
+    )
+    (pin "1")
+    (instances
+      (project "picoups"
+        (path "/d62f1157-7c2f-4dce-8167-d5624900d267"
+          (reference "TP4") (unit 1)
+        )
+        (path "/d62f1157-7c2f-4dce-8167-d5624900d267/69257c21-ade6-4c01-a27c-653d8ba74447"
+          (reference "TP2") (unit 1)
+        )
+      )
+    )
+  )
+  (symbol (lib_id "power:GND") (at 207.01 95.25 0) (mirror y) (unit 1)
+    (in_bom yes) (on_board yes) (dnp no) (fields_autoplaced)
+    (property "Reference" "#PWR033" (at 207.01 101.6 0)
+      (effects (font (size 1.27 1.27)) hide)
+    )
+    (property "Value" "GND" (at 207.01 99.06 90)
+      (effects (font (size 1.27 1.27)) (justify right))
+    )
+    (property "Footprint" "" (at 207.01 95.25 0)
+      (effects (font (size 1.27 1.27)) hide)
+    )
+    (property "Datasheet" "" (at 207.01 95.25 0)
+      (effects (font (size 1.27 1.27)) hide)
+    )
+    (pin "1")
+    (instances
+      (project "picoups"
+        (path "/d62f1157-7c2f-4dce-8167-d5624900d267"
+          (reference "#PWR033") (unit 1)
+        )
+      )
+    )
+  )
   (symbol (lib_id "power:GND") (at 57.15 137.16 270) (unit 1)
     (in_bom yes) (on_board yes) (dnp no) (fields_autoplaced)
@@
     )
   )
+  (symbol (lib_id "Connector:TestPoint") (at 180.34 92.71 0) (unit 1)
+    (in_bom yes) (on_board yes) (dnp no) (fields_autoplaced)
+    (property "Reference" "TP8" (at 182.88 88.138 0)
+      (effects (font (size 1.27 1.27)) (justify left))
+    )
+    (property "Value" "VBAT" (at 182.88 90.678 0)
+      (effects (font (size 1.27 1.27)) (justify left))
+    )
+    (property "Footprint" "TestPoint:TestPoint_Pad_D1.0mm" (at 185.42 92.71 0)
+      (effects (font (size 1.27 1.27)) hide)
+    )
+    (property "Datasheet" "~" (at 185.42 92.71 0)
+      (effects (font (size 1.27 1.27)) hide)
+    )
+    (pin "1")
+    (instances
+      (project "picoups"
+        (path "/d62f1157-7c2f-4dce-8167-d5624900d267"
+          (reference "TP8") (unit 1)
+        )
+        (path "/d62f1157-7c2f-4dce-8167-d5624900d267/69257c21-ade6-4c01-a27c-653d8ba74447"
+          (reference "TP2") (unit 1)
+        )
+      )
+    )
+  )
   (symbol (lib_id "power:GND") (at 60.96 41.91 0) (unit 1)
     (in_bom yes) (on_board yes) (dnp no) (fields_autoplaced)
@@
         (path "/d62f1157-7c2f-4dce-8167-d5624900d267"
           (reference "#PWR041") (unit 1)
+        )
+      )
+    )
+  )
+  (symbol (lib_id "power:GND") (at 189.23 95.25 0) (mirror y) (unit 1)
+    (in_bom yes) (on_board yes) (dnp no) (fields_autoplaced)
+    (property "Reference" "#PWR034" (at 189.23 101.6 0)
+      (effects (font (size 1.27 1.27)) hide)
+    )
+    (property "Value" "GND" (at 189.23 99.06 90)
+      (effects (font (size 1.27 1.27)) (justify right))
+    )
+    (property "Footprint" "" (at 189.23 95.25 0)
+      (effects (font (size 1.27 1.27)) hide)
+    )
+    (property "Datasheet" "" (at 189.23 95.25 0)
+      (effects (font (size 1.27 1.27)) hide)
+    )
+    (pin "1")
+    (instances
+      (project "picoups"
+        (path "/d62f1157-7c2f-4dce-8167-d5624900d267"
+          (reference "#PWR034") (unit 1)
         )
       )
@@
         )
       )
+    )
+  )
+  (symbol (lib_id "Connector:TestPoint") (at 198.12 92.71 0) (unit 1)
+    (in_bom yes) (on_board yes) (dnp no) (fields_autoplaced)
+    (property "Reference" "TP6" (at 200.66 88.138 0)
+      (effects (font (size 1.27 1.27)) (justify left))
+    )
+    (property "Value" "VBAT" (at 200.66 90.678 0)
+      (effects (font (size 1.27 1.27)) (justify left))
+    )
+    (property "Footprint" "TestPoint:TestPoint_Pad_D1.0mm" (at 203.2 92.71 0)
+      (effects (font (size 1.27 1.27)) hide)
+    )
+    (property "Datasheet" "~" (at 203.2 92.71 0)
+      (effects (font (size 1.27 1.27)) hide)
+    )
+    (pin "1")
+    (instances
+      (project "picoups"
+        (path "/d62f1157-7c2f-4dce-8167-d5624900d267"
+          (reference "TP6") (unit 1)
+        )
+        (path "/d62f1157-7c2f-4dce-8167-d5624900d267/69257c21-ade6-4c01-a27c-653d8ba74447"
+          (reference "TP2") (unit 1)
+        )
+      )

Commit message: Semi final v1.1
Parts:
- removed R15: 1M, Resistor_SMD:R_0805_2012Metric, symbol Device:R
Connections:
- net 3v3: no longer SW2.1
- net GND: now also SW2.1
- net SCL: now also JP1.1 (A), SW2.2
Changed lines of the file:
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@@
   (title_block
     (title "PicoUPS")
-    (date "2023-07-19")
-    (rev "1.0")
+    (date "2023-08-27")
+    (rev "1.1.0")
   )
   (junction (at 260.35 46.99) (diameter 0) (color 0 0 0 0)
@@
     (stroke (width 0) (type default))
   )
+  (wire (pts (xy 45.72 152.4) (xy 45.72 156.21))
+    (stroke (width 0) (type default))
+  )
   (wire (pts (xy 99.06 59.69) (xy 99.06 48.26))
     (stroke (width 0) (type default))
@@
     (stroke (width 0) (type default))
   )
+  (wire (pts (xy 45.72 152.4) (xy 49.53 152.4))
+    (stroke (width 0) (type default))
+  )
   (wire (pts (xy 107.95 102.87) (xy 111.76 102.87))
     (stroke (width 0) (type default))
@@
     (stroke (width 0) (type default))
   )
-  (wire (pts (xy 45.72 156.21) (xy 45.72 152.4))
-    (stroke (width 0) (type default))
-  )
-  (wire (pts (xy 45.72 163.83) (xy 45.72 167.64))
-    (stroke (width 0) (type default))
-  )
   (wire (pts (xy 273.05 46.99) (xy 275.59 46.99))
     (stroke (width 0) (type default))
@@
   )
   (wire (pts (xy 139.7 102.87) (xy 143.51 102.87))
-    (stroke (width 0) (type default))
-  )
-  (wire (pts (xy 45.72 152.4) (xy 49.53 152.4))
     (stroke (width 0) (type default))
   )
@@
     )
   )
+  (global_label "SCL" (shape bidirectional) (at 45.72 156.21 270) (fields_autoplaced)
+    (effects (font (size 1.27 1.27)) (justify right))
+    (property "Intersheetrefs" "${INTERSHEET_REFS}" (at 45.72 163.8141 90)
+      (effects (font (size 1.27 1.27)) (justify right) hide)
+    )
+  )
   (global_label "5V-" (shape passive) (at 215.9 95.25 270) (fields_autoplaced)
     (effects (font (size 1.27 1.27)) (justify right))
@@
     )
   )
-  (global_label "3v3" (shape input) (at 27.94 152.4 180) (fields_autoplaced)
-    (effects (font (size 1.27 1.27)) (justify right))
-    (property "Intersheetrefs" "${INTERSHEET_REFS}" (at 21.6476 152.4 0)
-      (effects (font (size 1.27 1.27)) (justify right) hide)
-    )
-  )
   (global_label "5V" (shape output) (at 275.59 46.99 0) (fields_autoplaced)
     (effects (font (size 1.27 1.27)) (justify left))
@@
     )
   )
-  (symbol (lib_id "power:GND") (at 45.72 167.64 0) (unit 1)
-    (in_bom yes) (on_board yes) (dnp no) (fields_autoplaced)
-    (property "Reference" "#PWR031" (at 45.72 173.99 0)
-      (effects (font (size 1.27 1.27)) hide)
-    )
-    (property "Value" "GND" (at 48.26 168.91 0)
-      (effects (font (size 1.27 1.27)) (justify left))
-    )
-    (property "Footprint" "" (at 45.72 167.64 0)
-      (effects (font (size 1.27 1.27)) hide)
-    )
-    (property "Datasheet" "" (at 45.72 167.64 0)
+  (symbol (lib_id "power:GND") (at 27.94 152.4 270) (unit 1)
+    (in_bom yes) (on_board yes) (dnp no) (fields_autoplaced)
+    (property "Reference" "#PWR031" (at 21.59 152.4 0)
+      (effects (font (size 1.27 1.27)) hide)
+    )
+    (property "Value" "GND" (at 24.13 152.4 90)
+      (effects (font (size 1.27 1.27)) (justify right))
+    )
+    (property "Footprint" "" (at 27.94 152.4 0)
+      (effects (font (size 1.27 1.27)) hide)
+    )
+    (property "Datasheet" "" (at 27.94 152.4 0)
       (effects (font (size 1.27 1.27)) hide)
     )
@@
         )
       )
-    )
-  )
-  (symbol (lib_id "Device:R") (at 45.72 160.02 180) (unit 1)
-    (in_bom yes) (on_board yes) (dnp no)
-    (property "Reference" "R15" (at 41.91 158.75 0)
-      (effects (font (size 1.27 1.27)))
-    )
-    (property "Value" "1M" (at 41.91 161.29 0)
-      (effects (font (size 1.27 1.27)))
-    )
-    (property "Footprint" "Resistor_SMD:R_0805_2012Metric" (at 47.498 160.02 90)
-      (effects (font (size 1.27 1.27)) hide)
-    )
-    (property "Datasheet" "~" (at 45.72 160.02 0)
-      (effects (font (size 1.27 1.27)) hide)
-    )
-    (pin "1")
-    (pin "2")
-    (instances
-      (project "picoups"
-        (path "/d62f1157-7c2f-4dce-8167-d5624900d267"
-          (reference "R15") (unit 1)
-        )
-        (path "/d62f1157-7c2f-4dce-8167-d5624900d267/92ed0473-53e9-4211-a651-f912f1c2bd2b"
-          (reference "R4") (unit 1)
-        )
-      )
