File: project/power_monitor.kicad_sch (KiCad schematic)
At the start: 2 parts

Commit message: Fixed mirrored RTC footprint
Parts:
- U?: footprint Package_DFN_QFN:Texas_RGV_S-PVQFN-N16_EP2.1x2.1mm -> Package_DFN_QFN:Texas_RGV_S-PVQFN-N16_EP2.1x2.1mm_ThermalVias
Changed lines of the file:
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@@
       (effects (font (size 1.27 1.27)) (justify left))
     )
-    (property "Footprint" "Package_DFN_QFN:Texas_RGV_S-PVQFN-N16_EP2.1x2.1mm" (at 149.86 72.39 0)
+    (property "Footprint" "Package_DFN_QFN:Texas_RGV_S-PVQFN-N16_EP2.1x2.1mm_ThermalVias" (at 149.86 72.39 0)
       (effects (font (size 1.27 1.27)) hide)
     )

Commit message: Final revision
Parts:
- gave numbers to parts that had none: 2
Changed lines of the file:
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@@
   (symbol (lib_id "power:GND") (at 170.18 91.44 0) (unit 1)
     (in_bom yes) (on_board yes) (dnp no) (fields_autoplaced)
-    (property "Reference" "#PWR?" (at 170.18 97.79 0)
+    (property "Reference" "#PWR016" (at 170.18 97.79 0)
       (effects (font (size 1.27 1.27)) hide)
     )
@@
     (instances
       (project "picoups"
-        (path "/d62f1157-7c2f-4dce-8167-d5624900d267"
-          (reference "#PWR?") (unit 1)
-        )
         (path "/d62f1157-7c2f-4dce-8167-d5624900d267/28cf3a3e-2270-4421-9985-b09e0cdb49a4"
           (reference "#PWR016") (unit 1)
@@
   (symbol (lib_id "power:GND") (at 147.32 119.38 0) (unit 1)
     (in_bom yes) (on_board yes) (dnp no) (fields_autoplaced)
-    (property "Reference" "#PWR?" (at 147.32 125.73 0)
+    (property "Reference" "#PWR012" (at 147.32 125.73 0)
       (effects (font (size 1.27 1.27)) hide)
     )
@@
     (instances
       (project "picoups"
-        (path "/d62f1157-7c2f-4dce-8167-d5624900d267"
-          (reference "#PWR?") (unit 1)
-        )
         (path "/d62f1157-7c2f-4dce-8167-d5624900d267/28cf3a3e-2270-4421-9985-b09e0cdb49a4"
           (reference "#PWR012") (unit 1)
@@
   (symbol (lib_id "Device:C") (at 170.18 85.09 0) (unit 1)
     (in_bom yes) (on_board yes) (dnp no) (fields_autoplaced)
-    (property "Reference" "C?" (at 173.99 83.82 0)
+    (property "Reference" "C11" (at 173.99 83.82 0)
       (effects (font (size 1.27 1.27)) (justify left))
     )
@@
     (instances
       (project "picoups"
-        (path "/d62f1157-7c2f-4dce-8167-d5624900d267"
-          (reference "C?") (unit 1)
-        )
         (path "/d62f1157-7c2f-4dce-8167-d5624900d267/28cf3a3e-2270-4421-9985-b09e0cdb49a4"
           (reference "C11") (unit 1)
@@
   (symbol (lib_id "Power_Management:INA3221") (at 149.86 100.33 0) (unit 1)
     (in_bom yes) (on_board yes) (dnp no) (fields_autoplaced)
-    (property "Reference" "U?" (at 154.3559 80.01 0)
+    (property "Reference" "U5" (at 154.3559 80.01 0)
       (effects (font (size 1.27 1.27)) (justify left))
     )
@@
     (instances
       (project "picoups"
-        (path "/d62f1157-7c2f-4dce-8167-d5624900d267"
-          (reference "U?") (unit 1)
-        )
         (path "/d62f1157-7c2f-4dce-8167-d5624900d267/28cf3a3e-2270-4421-9985-b09e0cdb49a4"
           (reference "U5") (unit 1)
@@
   (symbol (lib_id "power:GND") (at 152.4 78.74 180) (unit 1)
     (in_bom yes) (on_board yes) (dnp no) (fields_autoplaced)
-    (property "Reference" "#PWR?" (at 152.4 72.39 0)
+    (property "Reference" "#PWR013" (at 152.4 72.39 0)
       (effects (font (size 1.27 1.27)) hide)
     )
@@
     (instances
       (project "picoups"
-        (path "/d62f1157-7c2f-4dce-8167-d5624900d267"
-          (reference "#PWR?") (unit 1)
-        )
         (path "/d62f1157-7c2f-4dce-8167-d5624900d267/28cf3a3e-2270-4421-9985-b09e0cdb49a4"
           (reference "#PWR013") (unit 1)
@@
   (symbol (lib_id "power:GND") (at 166.37 111.76 0) (unit 1)
     (in_bom yes) (on_board yes) (dnp no) (fields_autoplaced)
-    (property "Reference" "#PWR?" (at 166.37 118.11 0)
+    (property "Reference" "#PWR015" (at 166.37 118.11 0)
       (effects (font (size 1.27 1.27)) hide)
     )
@@
     (instances
       (project "picoups"
-        (path "/d62f1157-7c2f-4dce-8167-d5624900d267"
-          (reference "#PWR?") (unit 1)
-        )
         (path "/d62f1157-7c2f-4dce-8167-d5624900d267/28cf3a3e-2270-4421-9985-b09e0cdb49a4"
           (reference "#PWR015") (unit 1)
@@
   (symbol (lib_id "power:GND") (at 152.4 119.38 0) (unit 1)
     (in_bom yes) (on_board yes) (dnp no) (fields_autoplaced)
-    (property "Reference" "#PWR?" (at 152.4 125.73 0)
+    (property "Reference" "#PWR014" (at 152.4 125.73 0)
       (effects (font (size 1.27 1.27)) hide)
     )
@@
     (instances
       (project "picoups"
-        (path "/d62f1157-7c2f-4dce-8167-d5624900d267"
-          (reference "#PWR?") (unit 1)
-        )
         (path "/d62f1157-7c2f-4dce-8167-d5624900d267/28cf3a3e-2270-4421-9985-b09e0cdb49a4"
           (reference "#PWR014") (unit 1)
