File: project/power_mux.kicad_sch (KiCad schematic)
At the start: 1 part, among them U6 TPS2116

Commit message: Added footprints
Parts:
- U6: footprint (none) -> Package_TO_SOT_SMD:SOT-583-8
Changed lines of the file:
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@@
       (effects (font (size 1.27 1.27)))
     )
-    (property "Footprint" "" (at 147.32 99.06 0)
+    (property "Footprint" "Package_TO_SOT_SMD:SOT-583-8" (at 147.32 99.06 0)
       (effects (font (size 1.27 1.27)) hide)
     )

Commit message: Final revision
Parts:
- renumbered U6 to U2
Changed lines of the file:
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@@
   (symbol (lib_id "PicoUPS:TPS2116") (at 147.32 99.06 0) (unit 1)
     (in_bom yes) (on_board yes) (dnp no)
-    (property "Reference" "U6" (at 147.32 87.63 0)
+    (property "Reference" "U2" (at 147.32 87.63 0)
       (effects (font (size 1.27 1.27)))
     )
@@
     (instances
       (project "picoups"
-        (path "/d62f1157-7c2f-4dce-8167-d5624900d267"
-          (reference "U6") (unit 1)
-        )
         (path "/d62f1157-7c2f-4dce-8167-d5624900d267/834bbbbe-6999-483a-a383-7c27b80d3fa6"
           (reference "U2") (unit 1)
@@
   (symbol (lib_id "power:GND") (at 160.02 102.87 90) (unit 1)
     (in_bom yes) (on_board yes) (dnp no) (fields_autoplaced)
-    (property "Reference" "#PWR039" (at 166.37 102.87 0)
+    (property "Reference" "#PWR022" (at 166.37 102.87 0)
       (effects (font (size 1.27 1.27)) hide)
     )
@@
     (instances
       (project "picoups"
-        (path "/d62f1157-7c2f-4dce-8167-d5624900d267"
-          (reference "#PWR039") (unit 1)
-        )
         (path "/d62f1157-7c2f-4dce-8167-d5624900d267/834bbbbe-6999-483a-a383-7c27b80d3fa6"
           (reference "#PWR022") (unit 1)
