File: project/usb_power_supply.kicad_sch (KiCad schematic)
At the start: 6 parts, among them U5 BQ24040

Commit message: Added symbol annotations
Other:
- moved on the sheet: C11
Changed lines of the file:
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@@
     (stroke (width 0) (type default))
   )
-  (wire (pts (xy 104.14 101.6) (xy 104.14 102.87))
+  (wire (pts (xy 101.6 101.6) (xy 101.6 102.87))
     (stroke (width 0) (type default))
   )
@@
     (stroke (width 0) (type default))
   )
-  (wire (pts (xy 104.14 92.71) (xy 104.14 93.98))
+  (wire (pts (xy 101.6 92.71) (xy 101.6 93.98))
     (stroke (width 0) (type default))
   )
@@
     (effects (font (size 1.27 1.27) bold) (justify left))
   )
-  (hierarchical_label "USB5V" (shape bidirectional) (at 104.14 92.71 90) (fields_autoplaced)
+  (hierarchical_label "USB5V" (shape bidirectional) (at 101.6 92.71 90) (fields_autoplaced)
     (effects (font (size 1.27 1.27) bold) (justify left))
   )
@@
   (symbol (lib_id "Device:R") (at 171.45 100.33 270) (mirror x) (unit 1)
     (in_bom yes) (on_board yes) (dnp no)
-    (property "Reference" "R16" (at 171.45 105.41 90)
-      (effects (font (size 1.27 1.27)))
-    )
-    (property "Value" "10k" (at 171.45 102.87 90)
+    (property "Reference" "R16" (at 171.45 102.87 90)
+      (effects (font (size 1.27 1.27)))
+    )
+    (property "Value" "10k" (at 171.45 105.41 90)
       (effects (font (size 1.27 1.27)))
     )
@@
         )
         (path "/d62f1157-7c2f-4dce-8167-d5624900d267/d2602436-7008-4d0c-96bd-d6a5c976935b"
-          (reference "R3") (unit 1)
+          (reference "R8") (unit 1)
         )
       )
@@
         )
         (path "/d62f1157-7c2f-4dce-8167-d5624900d267/d2602436-7008-4d0c-96bd-d6a5c976935b"
-          (reference "R1") (unit 1)
+          (reference "R6") (unit 1)
         )
       )
@@
         )
         (path "/d62f1157-7c2f-4dce-8167-d5624900d267/d2602436-7008-4d0c-96bd-d6a5c976935b"
-          (reference "U1") (unit 1)
+          (reference "U4") (unit 1)
         )
       )
@@
     )
   )
-  (symbol (lib_id "power:GND") (at 104.14 102.87 0) (unit 1)
+  (symbol (lib_id "power:GND") (at 101.6 102.87 0) (unit 1)
     (in_bom yes) (on_board yes) (dnp no) (fields_autoplaced)
-    (property "Reference" "#PWR037" (at 104.14 109.22 0)
-      (effects (font (size 1.27 1.27)) hide)
-    )
-    (property "Value" "GND" (at 104.14 107.95 0)
-      (effects (font (size 1.27 1.27)))
-    )
-    (property "Footprint" "" (at 104.14 102.87 0)
-      (effects (font (size 1.27 1.27)) hide)
-    )
-    (property "Datasheet" "" (at 104.14 102.87 0)
+    (property "Reference" "#PWR037" (at 101.6 109.22 0)
+      (effects (font (size 1.27 1.27)) hide)
+    )
+    (property "Value" "GND" (at 101.6 107.95 0)
+      (effects (font (size 1.27 1.27)))
+    )
+    (property "Footprint" "" (at 101.6 102.87 0)
+      (effects (font (size 1.27 1.27)) hide)
+    )
+    (property "Datasheet" "" (at 101.6 102.87 0)
       (effects (font (size 1.27 1.27)) hide)
     )
@@
   (symbol (lib_id "Device:R") (at 125.73 97.79 90) (mirror x) (unit 1)
     (in_bom yes) (on_board yes) (dnp no)
-    (property "Reference" "R13" (at 125.73 102.87 90)
-      (effects (font (size 1.27 1.27)))
-    )
-    (property "Value" "2k" (at 125.73 100.33 90)
+    (property "Reference" "R13" (at 125.73 100.33 90)
+      (effects (font (size 1.27 1.27)))
+    )
+    (property "Value" "2k" (at 125.73 102.87 90)
       (effects (font (size 1.27 1.27)))
     )
@@
         )
         (path "/d62f1157-7c2f-4dce-8167-d5624900d267/d2602436-7008-4d0c-96bd-d6a5c976935b"
-          (reference "R2") (unit 1)
-        )
-      )
-    )
-  )
-  (symbol (lib_id "Device:C") (at 104.14 97.79 0) (mirror x) (unit 1)
-    (in_bom yes) (on_board yes) (dnp no)
-    (property "Reference" "C11" (at 100.33 96.52 0)
-      (effects (font (size 1.27 1.27)) (justify right))
-    )
-    (property "Value" "1uF" (at 100.33 99.06 0)
-      (effects (font (size 1.27 1.27)) (justify right))
-    )
-    (property "Footprint" "Capacitor_SMD:C_0805_2012Metric" (at 105.1052 93.98 0)
-      (effects (font (size 1.27 1.27)) hide)
-    )
-    (property "Datasheet" "~" (at 104.14 97.79 0)
+          (reference "R7") (unit 1)
+        )
+      )
+    )
+  )
+  (symbol (lib_id "Device:C") (at 101.6 97.79 0) (mirror x) (unit 1)
+    (in_bom yes) (on_board yes) (dnp no)
+    (property "Reference" "C11" (at 105.41 96.52 0)
+      (effects (font (size 1.27 1.27)) (justify left))
+    )
+    (property "Value" "1uF" (at 105.41 99.06 0)
+      (effects (font (size 1.27 1.27)) (justify left))
+    )
+    (property "Footprint" "Capacitor_SMD:C_0805_2012Metric" (at 102.5652 93.98 0)
+      (effects (font (size 1.27 1.27)) hide)
+    )
+    (property "Datasheet" "~" (at 101.6 97.79 0)
       (effects (font (size 1.27 1.27)) hide)
     )
@@
         )
         (path "/d62f1157-7c2f-4dce-8167-d5624900d267/d2602436-7008-4d0c-96bd-d6a5c976935b"
-          (reference "C1") (unit 1)
+          (reference "C9") (unit 1)
         )
       )
@@
         )
         (path "/d62f1157-7c2f-4dce-8167-d5624900d267/d2602436-7008-4d0c-96bd-d6a5c976935b"
-          (reference "C2") (unit 1)
-        )
-      )
+          (reference "C10") (unit 1)
+        )
+      )

Commit message: Added footprints
Parts:
- U5: footprint (none) -> Package_SON:WSON-6_1.5x1.5mm_P0.5mm
Changed lines of the file:
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@@
       (effects (font (size 1.27 1.27)))
     )
-    (property "Footprint" "" (at 148.59 97.79 0)
+    (property "Footprint" "Package_SON:WSON-6_1.5x1.5mm_P0.5mm" (at 148.59 97.79 0)
       (effects (font (size 1.27 1.27)) hide)
     )

Commit message: Fix BQ2404 footprint
Parts:
- U5: footprint Package_SON:WSON-6_1.5x1.5mm_P0.5mm -> PicoUPS:WSON-10-1EP_2x2mm_P0.5mm
Changed lines of the file:
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@@
       (effects (font (size 1.27 1.27)))
     )
-    (property "Footprint" "Package_SON:WSON-6_1.5x1.5mm_P0.5mm" (at 148.59 97.79 0)
+    (property "Footprint" "PicoUPS:WSON-10-1EP_2x2mm_P0.5mm" (at 148.59 97.79 0)
       (effects (font (size 1.27 1.27)) hide)
     )

Commit message: Fixed solar status LEDs wrong VBAT
Connections:
- net GND: now also U5.11 (GND)
Changed lines of the file:
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@@
     (pin "1")
     (pin "10")
+    (pin "11")
     (pin "2")
     (pin "3")

Commit message: Final revision
Parts:
- renumbered C9 to C10, C11 to C9, R12 to R6, R13 to R7, R16 to R8, U5 to U4
Changed lines of the file:
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@@
   (symbol (lib_id "Device:R") (at 171.45 100.33 270) (mirror x) (unit 1)
     (in_bom yes) (on_board yes) (dnp no)
-    (property "Reference" "R16" (at 171.45 102.87 90)
+    (property "Reference" "R8" (at 171.45 102.87 90)
       (effects (font (size 1.27 1.27)))
     )
@@
     (instances
       (project "picoups"
-        (path "/d62f1157-7c2f-4dce-8167-d5624900d267"
-          (reference "R16") (unit 1)
-        )
         (path "/d62f1157-7c2f-4dce-8167-d5624900d267/d2602436-7008-4d0c-96bd-d6a5c976935b"
           (reference "R8") (unit 1)
@@
   (symbol (lib_id "Device:R") (at 125.73 95.25 90) (unit 1)
     (in_bom yes) (on_board yes) (dnp no)
-    (property "Reference" "R12" (at 125.73 90.17 90)
+    (property "Reference" "R6" (at 125.73 90.17 90)
       (effects (font (size 1.27 1.27)))
     )
@@
     (instances
       (project "picoups"
-        (path "/d62f1157-7c2f-4dce-8167-d5624900d267"
-          (reference "R12") (unit 1)
-        )
         (path "/d62f1157-7c2f-4dce-8167-d5624900d267/d2602436-7008-4d0c-96bd-d6a5c976935b"
           (reference "R6") (unit 1)
@@
   (symbol (lib_id "power:GND") (at 119.38 97.79 270) (unit 1)
     (in_bom yes) (on_board yes) (dnp no) (fields_autoplaced)
-    (property "Reference" "#PWR034" (at 113.03 97.79 0)
+    (property "Reference" "#PWR06" (at 113.03 97.79 0)
       (effects (font (size 1.27 1.27)) hide)
     )
@@
     (instances
       (project "picoups"
-        (path "/d62f1157-7c2f-4dce-8167-d5624900d267"
-          (reference "#PWR034") (unit 1)
-        )
         (path "/d62f1157-7c2f-4dce-8167-d5624900d267/d2602436-7008-4d0c-96bd-d6a5c976935b"
           (reference "#PWR06") (unit 1)
@@
   (symbol (lib_id "PicoUPS:BQ24040") (at 148.59 97.79 0) (unit 1)
     (in_bom yes) (on_board yes) (dnp no)
-    (property "Reference" "U5" (at 148.59 85.09 0)
+    (property "Reference" "U4" (at 148.59 85.09 0)
       (effects (font (size 1.27 1.27)))
     )
@@
     (instances
       (project "picoups"
-        (path "/d62f1157-7c2f-4dce-8167-d5624900d267"
-          (reference "U5") (unit 1)
-        )
         (path "/d62f1157-7c2f-4dce-8167-d5624900d267/d2602436-7008-4d0c-96bd-d6a5c976935b"
           (reference "U4") (unit 1)
@@
   (symbol (lib_id "power:GND") (at 119.38 95.25 270) (unit 1)
     (in_bom yes) (on_board yes) (dnp no) (fields_autoplaced)
-    (property "Reference" "#PWR033" (at 113.03 95.25 0)
+    (property "Reference" "#PWR03" (at 113.03 95.25 0)
       (effects (font (size 1.27 1.27)) hide)
     )
@@
     (instances
       (project "picoups"
-        (path "/d62f1157-7c2f-4dce-8167-d5624900d267"
-          (reference "#PWR033") (unit 1)
-        )
         (path "/d62f1157-7c2f-4dce-8167-d5624900d267/d2602436-7008-4d0c-96bd-d6a5c976935b"
           (reference "#PWR03") (unit 1)
@@
   (symbol (lib_id "power:GND") (at 101.6 102.87 0) (unit 1)
     (in_bom yes) (on_board yes) (dnp no) (fields_autoplaced)
-    (property "Reference" "#PWR037" (at 101.6 109.22 0)
+    (property "Reference" "#PWR02" (at 101.6 109.22 0)
       (effects (font (size 1.27 1.27)) hide)
     )
@@
     (instances
       (project "picoups"
-        (path "/d62f1157-7c2f-4dce-8167-d5624900d267"
-          (reference "#PWR037") (unit 1)
-        )
         (path "/d62f1157-7c2f-4dce-8167-d5624900d267/d2602436-7008-4d0c-96bd-d6a5c976935b"
           (reference "#PWR02") (unit 1)
@@
   (symbol (lib_id "Device:R") (at 125.73 97.79 90) (mirror x) (unit 1)
     (in_bom yes) (on_board yes) (dnp no)
-    (property "Reference" "R13" (at 125.73 100.33 90)
+    (property "Reference" "R7" (at 125.73 100.33 90)
       (effects (font (size 1.27 1.27)))
     )
@@
     (instances
       (project "picoups"
-        (path "/d62f1157-7c2f-4dce-8167-d5624900d267"
-          (reference "R13") (unit 1)
-        )
         (path "/d62f1157-7c2f-4dce-8167-d5624900d267/d2602436-7008-4d0c-96bd-d6a5c976935b"
           (reference "R7") (unit 1)
@@
   (symbol (lib_id "Device:C") (at 101.6 97.79 0) (mirror x) (unit 1)
     (in_bom yes) (on_board yes) (dnp no)
-    (property "Reference" "C11" (at 105.41 96.52 0)
+    (property "Reference" "C9" (at 105.41 96.52 0)
       (effects (font (size 1.27 1.27)) (justify left))
     )
@@
     (instances
       (project "picoups"
-        (path "/d62f1157-7c2f-4dce-8167-d5624900d267"
-          (reference "C11") (unit 1)
-        )
         (path "/d62f1157-7c2f-4dce-8167-d5624900d267/d2602436-7008-4d0c-96bd-d6a5c976935b"
           (reference "C9") (unit 1)
@@
   (symbol (lib_id "Device:C") (at 193.04 97.79 0) (unit 1)
     (in_bom yes) (on_board yes) (dnp no) (fields_autoplaced)
-    (property "Reference" "C9" (at 196.85 96.52 0)
+    (property "Reference" "C10" (at 196.85 96.52 0)
       (effects (font (size 1.27 1.27)) (justify left))
     )
@@
     (instances
       (project "picoups"
-        (path "/d62f1157-7c2f-4dce-8167-d5624900d267"
-          (reference "C9") (unit 1)
-        )
         (path "/d62f1157-7c2f-4dce-8167-d5624900d267/d2602436-7008-4d0c-96bd-d6a5c976935b"
           (reference "C10") (unit 1)
@@
   (symbol (lib_id "power:GND") (at 148.59 111.76 0) (unit 1)
     (in_bom yes) (on_board yes) (dnp no) (fields_autoplaced)
-    (property "Reference" "#PWR035" (at 148.59 118.11 0)
+    (property "Reference" "#PWR08" (at 148.59 118.11 0)
       (effects (font (size 1.27 1.27)) hide)
     )
@@
     (instances
       (project "picoups"
-        (path "/d62f1157-7c2f-4dce-8167-d5624900d267"
-          (reference "#PWR035") (unit 1)
-        )
         (path "/d62f1157-7c2f-4dce-8167-d5624900d267/d2602436-7008-4d0c-96bd-d6a5c976935b"
           (reference "#PWR08") (unit 1)
@@
   (symbol (lib_id "power:GND") (at 193.04 102.87 0) (unit 1)
     (in_bom yes) (on_board yes) (dnp no) (fields_autoplaced)
-    (property "Reference" "#PWR038" (at 193.04 109.22 0)
+    (property "Reference" "#PWR010" (at 193.04 109.22 0)
       (effects (font (size 1.27 1.27)) hide)
     )
@@
     (instances
       (project "picoups"
-        (path "/d62f1157-7c2f-4dce-8167-d5624900d267"
-          (reference "#PWR038") (unit 1)
-        )
         (path "/d62f1157-7c2f-4dce-8167-d5624900d267/d2602436-7008-4d0c-96bd-d6a5c976935b"
           (reference "#PWR010") (unit 1)
@@
   (symbol (lib_id "power:GND") (at 179.07 100.33 90) (unit 1)
     (in_bom yes) (on_board yes) (dnp no) (fields_autoplaced)
-    (property "Reference" "#PWR036" (at 185.42 100.33 0)
+    (property "Reference" "#PWR09" (at 185.42 100.33 0)
       (effects (font (size 1.27 1.27)) hide)
     )
@@
     (instances
       (project "picoups"
-        (path "/d62f1157-7c2f-4dce-8167-d5624900d267"
-          (reference "#PWR036") (unit 1)
-        )
         (path "/d62f1157-7c2f-4dce-8167-d5624900d267/d2602436-7008-4d0c-96bd-d6a5c976935b"
           (reference "#PWR09") (unit 1)
@@
   (symbol (lib_id "power:GND") (at 130.81 102.87 0) (unit 1)
     (in_bom yes) (on_board yes) (dnp no) (fields_autoplaced)
-    (property "Reference" "#PWR031" (at 130.81 109.22 0)
+    (property "Reference" "#PWR07" (at 130.81 109.22 0)
       (effects (font (size 1.27 1.27)) hide)
     )
@@
     (instances
       (project "picoups"
-        (path "/d62f1157-7c2f-4dce-8167-d5624900d267"
-          (reference "#PWR031") (unit 1)
-        )
         (path "/d62f1157-7c2f-4dce-8167-d5624900d267/d2602436-7008-4d0c-96bd-d6a5c976935b"
           (reference "#PWR07") (unit 1)
